File: Ki-Cad files/Fi-Pad.kicad_pcb (KiCad board)
At the start: 2 copper layers, 89.3 x 66.1 mm, 15 parts, among them J1 0.91 Oled Display, SW1 Mx-Switch, SW2 Mx-Switch, SW3 Mx-Switch, SW4 Mx-Switch, SW5 Mx-Switch, SW6 Mx-Switch, SW7 Mx-Switch, SW8 Mx-Switch, SW9 Mx-Switch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

Commit message: Updating Ki-CAD files
Connections:
- U1 pad 12: unconnected-(U1-3V3-Pad12) -> Net-(J1-Pin_2)
- U1 pad 14: Net-(J1-Pin_2) -> unconnected-(U1-5V-Pad14)
Routing:
- net GND: track 221.3 -> 242.8 mm
- net Net-(J1-Pin_2): track 0.00 -> 11.0 mm
Changed lines of the file:
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@@
 			(outputformat 1)
 			(mirror no)
-			(drillshape 1)
+			(drillshape 0)
 			(scaleselection 1)
-			(outputdirectory "")
+			(outputdirectory "../")
 		)
 	)
@@
 	(net 15 "unconnected-(U1-BAT-Pad15)")
 	(net 16 "unconnected-(U1-SWDCLK-Pad18)")
-	(net 17 "unconnected-(U1-3V3-Pad12)")
+	(net 17 "unconnected-(U1-5V-Pad14)")
 	(net 18 "unconnected-(U1-RST-Pad19)")
 	(footprint "PCM_Switch_Keyboard_Cherry_MX:SW_Cherry_MX_PCB_1.00u"
@@
 			(layers "F.Cu" "F.Mask" "F.Paste")
 			(roundrect_rratio 0.25)
-			(net 17 "unconnected-(U1-3V3-Pad12)")
+			(net 2 "Net-(J1-Pin_2)")
 			(pinfunction "3V3")
-			(pintype "passive+no_connect")
+			(pintype "passive")
 			(solder_mask_margin 0.0508)
 			(thermal_bridge_angle 45)
@@
 			(layers "F.Cu" "F.Mask" "F.Paste")
 			(roundrect_rratio 0.25)
-			(net 2 "Net-(J1-Pin_2)")
+			(net 17 "unconnected-(U1-5V-Pad14)")
 			(pinfunction "5V")
-			(pintype "passive")
+			(pintype "passive+no_connect")
 			(solder_mask_margin 0.0508)
 			(thermal_bridge_angle 45)
@@
 	(dimension
 		(type orthogonal)
-		(layer "Edge.Cuts")
+		(layer "User.1")
 		(pts
 			(xy 196.32 68.6) (xy 107.02 72.6)
@@
 		(gr_text "89.3"
 			(at 151.67 58.05 0)
-			(layer "Edge.Cuts")
+			(layer "User.1")
 			(effects
 				(font
@@
 	(dimension
 		(type orthogonal)
-		(layer "Edge.Cuts")
+		(layer "User.1")
 		(pts
 			(xy 188.92 131) (xy 185.42 64.9)
@@
 		(gr_text "66.1"
 			(at 200.47 97.95 90)
-			(layer "Edge.Cuts")
+			(layer "User.1")
 			(effects
 				(font
@@
 	)
 	(segment
+		(start 115.62 89.195)
+		(end 114.88 89.935)
+		(width 0.2)
+		(layer "F.Cu")
+		(net 2)
+	)
+	(segment
+		(start 115.62 79.2)
+		(end 115.62 89.195)
+		(width 0.2)
+		(layer "F.Cu")
+		(net 2)
+	)
+	(segment
 		(start 122.5 106.1)
 		(end 122.5 109.08)
@@
 	)
 	(segment
+		(start 126.06 96.648)
+		(end 111.582 96.648)
+		(width 0.2)
+		(layer "F.Cu")
+		(net 4)
+	)
+	(segment
 		(start 112.32 89.915)
 		(end 112.34 89.935)
@@
 	)
 	(segment
+		(start 111.582 96.648)
+		(end 111.582 90.693)
+		(width 0.2)
+		(layer "F.Cu")
+		(net 4)
+	)
+	(segment
 		(start 188.62 75.9)
 		(end 188.62 89.8)
@@
 		(width 0.2)
 		(layer "F.Cu")
+		(net 4)
+	)
+	(segment
+		(start 111.582 90.693)
+		(end 112.34 89.935)
+		(width 0.2)
+		(layer "F.Cu")
