File: Ki-Cad files/Fi-Pad.kicad_sch (KiCad schematic)
At the start: 11 parts, among them J1 0.91 Oled Display, SW1 Mx-Switch, SW2 Mx-Switch, SW3 Mx-Switch, SW4 Mx-Switch, SW5 Mx-Switch, SW6 Mx-Switch, SW7 Mx-Switch, SW8 Mx-Switch, SW9 Mx-Switch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

Commit message: Updating Ki-CAD files
Connections:
- net at J1.2 (Pin_2): now also U1.12 (3V3); no longer U1.14 (5V)
Changed lines of the file:
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@@
-	)
-	(no_connect
-		(at 99.06 57.15)
 	)
 	(no_connect
@@
 		(at 80.01 76.2)
 	)
+	(no_connect
+		(at 91.44 57.15)
+	)
 	(wire
 		(pts
@@
 	(wire
 		(pts
-			(xy 67.31 52.07) (xy 91.44 52.07)
+			(xy 67.31 44.45) (xy 99.06 44.45)
 		)
 		(stroke
@@
 	(wire
 		(pts
+			(xy 99.06 44.45) (xy 99.06 57.15)
+		)
+		(stroke
+			(width 0)
+			(type default)
+		)
+	)
+	(wire
+		(pts
 			(xy 104.14 114.3) (xy 67.31 114.3)
 		)
@@
 	(wire
 		(pts
-			(xy 91.44 52.07) (xy 91.44 57.15)
-		)
-		(stroke
-			(width 0)
-			(type default)
-		)
-	)
-	(wire
-		(pts
 			(xy 149.86 83.82) (xy 154.94 83.82)
 		)
@@
 	(wire
 		(pts
-			(xy 67.31 114.3) (xy 67.31 52.07)
-		)
-		(stroke
+			(xy 67.31 114.3) (xy 67.31 44.45)
+		)
+		(stroke
